Commit message: fix mesh

File: lingao_description_ros2/urdf/MiniUGV_10A.xacro (robot description, xacro)
@@ -13,5 +13,5 @@
         <origin xyz="0 0 0" rpy="0 0 0" />
         <geometry>
-            <mesh filename="package://lingao_description/meshes/LA_MiniUGV_10A/mobile_base.stl" scale="1 1 1"/>
+            <mesh filename="file://$(find lingao_description_ros2)/meshes/LA_MiniUGV_10A/mobile_base.stl" scale="1 1 1"/>
         </geometry>
         <material name="yellow">
@@ -44,5 +44,5 @@
                 <origin xyz="0 0 0" rpy="0 0 0" />
                 <geometry>
-                    <mesh filename="package://lingao_description/meshes/LA_MiniUGV_10A/mobile_whell.stl" />
+                    <mesh filename="file://$(find lingao_description_ros2)/meshes/LA_MiniUGV_10A/mobile_whell.stl" />
                 </geometry>
                 <material name="Poppy">
@@ -64,5 +64,5 @@
             </inertial>
         </link>
-        <joint name="${link_name}_wheel" type="fixed">
+        <joint name="${link_name}_wheel" type="continuous">
             <parent link="${parent_link}"/>
             <child link="${link_name}_wheel_link"/>
