Commit message: add gazebo launch

File: lingao_description/urdf/MiniUGV_10A.xacro (robot description, xacro)
@@ -1,42 +1,54 @@
 <?xml version="1.0"?>
 <robot name="MiniUGV_10A" xmlns:xacro="http://ros.org/wiki/xacro">
-    <!--property list -->
+    <!-- basic shapes -->
+    <xacro:include filename="$(find urdf_basic_shapes)/urdf/basic_shapes.urdf.xacro" />
+    <!-- basic inertia -->
+    <!-- <xacro:include filename="$(find urdf_basic_shapes)/urdf/inertia.urdf.xacro" /> -->
+    <!--property
+    list -->
     <xacro:property name="M_PI" value="3.1415926535897931" />
-    <xacro:property name="base_mass"   value="20" />
-    <xacro:property name="base_length" value="0.445"/>
-    <xacro:property name="base_width" value="0.345"/>
-    <xacro:property name="base_height" value="0.184"/>
+    <xacro:property name="base_mass" value="20" />
+    <xacro:property name="base_length" value="0.445" />
+    <xacro:property name="base_width" value="0.345" />
+    <xacro:property name="base_height" value="0.184" />
     <xacro:property name="earth_space" value="0.055" />
     <!-- Base link -->
     <link name="base_link">
-      <visual>
-        <origin xyz="0 0 0" rpy="0 0 0" />
-        <geometry>
-            <mesh filename="file://$(find lingao_description_ros2)/meshes/LA_MiniUGV_10A/mobile_base.stl" scale="1 1 1"/>
-        </geometry>
-        <material name="yellow">
-          <color rgba="1.0 0.812 0.0 1.0" />
-        </material>
-      </visual>
-      <collision>
+        <visual>
             <origin xyz="0 0 0" rpy="0 0 0" />
             <geometry>
-                <box size="${base_length} ${base_width} ${base_height}"/>
+                <!-- <box size="${base_length} ${base_width} ${base_height}" /> -->
+                <mesh
+                    filename="file://$(find lingao_description_ros2)/meshes/LA_MiniUGV_10A/mobile_base.stl"
+                    scale="1 1 1" />
+            </geometry>
+            <material name="yellow">
+                <color rgba="1.0 0.812 0.0 1.0" />
+            </material>
+        </visual>
+        <collision>
+            <origin xyz="0 0 ${earth_space}" rpy="0 0 0" />
+            <geometry>
+                <box size="${base_length} ${base_width} ${base_height}" />
             </geometry>
         </collision>
+        <xacro:solid_cuboid_inertia m="${base_mass}" h="${base_height}" d="${base_length}"
+            w="${base_width}" />
     </link>
-    <link name="base_footprint"/>
+    <xacro:gazebo_params name="base_link" rgb="Yellow"
+        friction="${sliding_friction}" />
+    <link name="base_footprint" />
     <joint name="base_footprint_joint" type="fixed">
-      <parent link="base_footprint" />
-      <child link="base_link" />
-      <origin xyz="0 0 ${earth_space}" />
+        <parent link="base_footprint" />
+        <child link="base_link" />
+        <origin xyz="0 0 ${earth_space}" />
     </joint>
     <!-- WHELL -->
-    <xacro:property name="wheel_radius" value="0.0325" />
-    <xacro:property name="wheel_length" value="0.0152" />
-    <xacro:property name="wheel_base"   value="0.24"/>
-    <xacro:property name="wheel_track"  value="0.333"/>
-    <xacro:property name="wheel_joint_z"  value="0.02"/>
-    <xacro:property name="wheel_mass"   value="1" />
+    <xacro:property name="wheel_radius" value="0.075" />
+    <xacro:property name="wheel_length" value="0.03" />
+    <xacro:property name="wheel_base" value="0.24" />
+    <xacro:property name="wheel_track" value="0.333" />
+    <xacro:property name="wheel_joint_z" value="0.02" />
+    <xacro:property name="wheel_mass" value="1" />
     <xacro:macro name="base_wheel" params="link_name parent_link reflect mass *joint_pose">
         <link name="${link_name}_wheel_link">
@@ -44,35 +56,42 @@
                 <origin xyz="0 0 0" rpy="0 0 0" />
                 <geometry>
-                    <mesh filename="file://$(find lingao_description_ros2)/meshes/LA_MiniUGV_10A/mobile_whell.stl" />
+                    <!-- <cylinder length="${wheel_length}" radius="${wheel_radius}" /> -->
+                    <mesh
+                        filename="file://$(find lingao_description_ros2)/meshes/LA_MiniUGV_10A/mobile_whell.stl" />
                 </geometry>
                 <material name="Poppy">
-                    <color rgba="0.4 0.4039 0.42745098 1.0"/>
+                    <color rgba="0.4 0.4039 0.42745098 1.0" />
                 </material>
             </visual>
             <collision>
-              <origin xyz="0 ${wheel_length/2} 0" rpy="${pi/2} 0 0" />
-              <geometry>
-                  <cylinder length="${wheel_length}" radius="${wheel_radius}" />
-              </geometry>
+                <origin xyz="0 ${wheel_length/2} 0" rpy="${pi/2} 0 0" />
+                <geometry>
+                    <sphere radius="${wheel_radius}" />
+                    <!-- </geometry> length="${wheel_length}" radius="${wheel_radius}" /> -->
+                </geometry>
             </collision>
             <inertial>
-                <origin xyz="0 0 0" rpy="0 0 0"/>
-                <mass value="${mass}"/>
+                <origin xyz="0 0 0" rpy="0 0 0" />
+                <mass value="${mass}" />
                 <inertia ixx="${(2/5) * mass * (wheel_radius * wheel_radius)}" ixy="0" ixz="0"
-                        iyy="${(2/5) * mass * (wheel_radius * wheel_radius)}" iyz="0"
-                        izz="${(2/5) * mass * (wheel_radius * wheel_radius)}" />
+                    iyy="${(2/5) * mass * (wheel_radius * wheel_radius)}" iyz="0"
+                    izz="${(2/5) * mass * (wheel_radius * wheel_radius)}" />
             </inertial>
         </link>
+        <xacro:gazebo_params name="${link_name}_wheel_link" rgb="Grey"
+            friction="${sliding_friction}" />
         <joint name="${link_name}_wheel" type="continuous">
-            <parent link="${parent_link}"/>
-            <child link="${link_name}_wheel_link"/>
-            <xacro:insert_block name="joint_pose"/>
-            <axis xyz="0 ${reflect*1} 0"/>
+            <parent link="${parent_link}" />
+            <child link="${link_name}_wheel_link" />
+            <xacro:insert_block name="joint_pose" />
+            <axis xyz="0 ${reflect*1} 0" />
         </joint>
     </xacro:macro>
-    <xacro:base_wheel parent_link="base_link" link_name="front_left" reflect="1" mass="${wheel_mass}">
+    <xacro:base_wheel parent_link="base_link" link_name="front_left" reflect="1"
+        mass="${wheel_mass}">
         <origin xyz="${wheel_base/2} ${wheel_track/2} ${wheel_joint_z}" rpy="0 0 0" />
     </xacro:base_wheel>
-    <xacro:base_wheel parent_link="base_link" link_name="front_right" reflect="-1" mass="${wheel_mass}">
+    <xacro:base_wheel parent_link="base_link" link_name="front_right" reflect="-1"
+        mass="${wheel_mass}">
         <origin xyz="${wheel_base/2} ${-wheel_track/2} ${wheel_joint_z}" rpy="0 0 ${M_PI}" />
     </xacro:base_wheel>
@@ -80,6 +99,17 @@
         <origin xyz="${-wheel_base/2} ${wheel_track/2} ${wheel_joint_z}" rpy="0 0 0" />
     </xacro:base_wheel>
-    <xacro:base_wheel parent_link="base_link" link_name="rear_right" reflect="-1" mass="${wheel_mass}">
+    <xacro:base_wheel parent_link="base_link" link_name="rear_right" reflect="-1"
+        mass="${wheel_mass}">
         <origin xyz="${-wheel_base/2} ${-wheel_track/2} ${wheel_joint_z}" rpy="0 0 ${M_PI}" />
     </xacro:base_wheel>
+    <!-- Skid Steering Drive -->
+    <gazebo>
+        <plugin name="object_controller" filename="libgazebo_ros_planar_move.so">
+            <commandTopic>cmd_vel</commandTopic>
+            <odometryTopic>odom</odometryTopic>
+            <odometryFrame>odom</odometryFrame>
+            <odometryRate>20.0</odometryRate>
+            <robotBaseFrame>base_footprint</robotBaseFrame>
+        </plugin>
+    </gazebo>
 </robot>
